File: motor_control_board/PWR.kicad_sch (KiCad schematic)
At the start: 17 parts, among them Q1 ECH8420-TL-H, U6 SN74LVC1G14DBV, U7 INA232AIDDFR, U8 UA78M05IDCYR

Commit message: PCB routing 70% done
Parts:
- removed Q1: ECH8420-TL-H, Package_TO_SOT_SMD:OnSemi_ECH8, symbol canhw:NMOS
- added U9: ECH8420-TL-H, Package_TO_SOT_SMD:OnSemi_ECH8, symbol ECH8420-TL-H:ECH8420-TL-H
Connections:
- net GND: now also U9.1 (SOURCE), U9.2 (SOURCE), U9.3 (SOURCE)
- net Servo-: now also U9.5 (DRAIN), U9.6 (DRAIN), U9.7 (DRAIN), U9.8 (DRAIN)
- net at R24.2: now also U9.4 (GATE)

Commit message: Routing Complete
Connections:
- net LDO_OUT: now reaches C14.1, F3.2, U8.3 (OUTPUT)
Changed lines of the file:
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@@
+		)
+	)
+	(label "LDO_OUT"
+		(at 200.025 100.965 0)
+		(fields_autoplaced yes)
+		(effects
+			(font
+				(size 1.27 1.27)
+			)
+			(justify left bottom)
 		)
 	)

Commit message: Fixed symbol and footprint libraries
Parts:
- U9: symbol ECH8420-TL-H:ECH8420-TL-H -> canhw:ECH8420-TL-H
Changed lines of the file:
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@@
 	)
 	(symbol
-		(lib_id "ECH8420-TL-H:ECH8420-TL-H")
+		(lib_id "canhw:ECH8420-TL-H")
 		(at 140.97 149.86 0)
 		(unit 1)

Commit message: Fixed DRC errors except for the PTH keep out zones
Parts:
- U7: footprint motor-control:SOT65P280X110-8N -> canhw_footprints:SOT65P280X110-8N
- U8: footprint motor-control:SOT230P700X180-4N -> canhw_footprints:SOT230P700X180-4N
Changed lines of the file:
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@@
 			)
 		)
-		(property "Footprint" "motor-control:SOT230P700X180-4N"
+		(property "Footprint" "canhw_footprints:SOT230P700X180-4N"
 			(at 235.585 114.935 0)
 			(effects
@@
 			)
 		)
-		(property "Footprint" "motor-control:SOT65P280X110-8N"
+		(property "Footprint" "canhw_footprints:SOT65P280X110-8N"
 			(at 128.27 76.2 0)
 			(effects
