File: motor_control_board/PWR.kicad_sch (KiCad schematic)
At the start: 17 parts, among them U6 SN74LVC1G14DBV, U7 INA232AIDDFR, U8 UA78M05IDCYR, U9 ECH8420-TL-H

Commit message: Fix DRC warnings
Changed lines of the file:
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@@
-	)
-	(junction
-		(at 191.135 139.065)
-		(diameter 0)
-		(color 0 0 0 0)
 	)
 	(junction
@@
 		(pts
 			(xy 191.135 139.065) (xy 191.135 149.86)
-		)
-		(stroke
-			(width 0)
-			(type default)
-		)
-	)
-	(wire
-		(pts
-			(xy 191.135 135.255) (xy 191.135 139.065)
 		)
 		(stroke
@@
 					(unit 1)
 				)
-			)
-		)
-	)
-	(symbol
-		(lib_id "canhw:PWR_FLAG")
-		(at 191.135 135.255 0)
-		(unit 1)
-		(exclude_from_sim no)
-		(in_bom yes)
-		(on_board yes)
-		(dnp no)
-		(fields_autoplaced yes)
-		(property "Reference" "#FLG01"
-			(at 191.135 133.35 0)
-			(effects
-				(font
-					(size 1.27 1.27)
-				)
-				(hide yes)
-			)
-		)
-		(property "Value" "PWR_FLAG"
-			(at 191.135 130.175 0)
-			(effects
-				(font
-					(size 1.27 1.27)
-				)
-			)
-		)
-		(property "Footprint" ""
-			(at 191.135 135.255 0)
-			(effects
-				(font
-					(size 1.27 1.27)
-				)
-				(hide yes)
-			)
-		)
-		(property "Datasheet" "~"
-			(at 191.135 135.255 0)
-			(effects
-				(font
-					(size 1.27 1.27)
-				)
-				(hide yes)
-			)
-		)
-		(property "Description" "Special symbol for telling ERC where power comes from"
-			(at 191.135 135.255 0)
-			(effects
-				(font
-					(size 1.27 1.27)
-				)
-				(hide yes)
-			)
-		)
-		(pin "1"
-		)
-		(instances
-			(project ""
-				(path "/ced26b11-410b-4897-bfe1-68b095b3fef4/6d921c46-a69c-4b88-8fde-0dba583b7bde"
-					(reference "#FLG01")
-					(unit 1)
-				)

Commit message: Address concerns
Parts:
- F3: value Polyfuse 1A -> Polyfuse 0.5A
Changed lines of the file:
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@@
 			)
 		)
-		(property "Value" "Polyfuse 1A"
+		(property "Value" "Polyfuse 0.5A"
 			(at 202.565 95.885 0)
 			(effects

Commit message: addressed concerns
Connections:
- net LDO_OUT: no longer names the net of C14.1, F3.2, U8.3 (OUTPUT)
Changed lines of the file:
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@@
-		)
-	)
-	(label "LDO_OUT"
-		(at 200.025 100.965 0)
-		(fields_autoplaced yes)
-		(effects
-			(font
-				(size 1.27 1.27)
-			)
-			(justify left bottom)
 		)
 	)
